File: Chromesthesia.kicad_pcb (KiCad board)
At the start: 2 copper layers, 164 x 105 mm, 577 parts

Commit message: Initial Production
Parts:
- added H1: MountingHole, MountingHole:MountingHole_2.2mm_M2, F.Cu at (209.2, 69.1)
- added H2: MountingHole, MountingHole:MountingHole_2.2mm_M2, F.Cu at (99.8, 69.2)
- added H3: MountingHole, MountingHole:MountingHole_2.2mm_M2, F.Cu at (99.8, 143.2)
- added H4: MountingHole, MountingHole:MountingHole_2.2mm_M2, F.Cu at (209.2, 143.2)
- added J3: Interface, Connector_JST:JST_VH_B4P-VH-FB-B_1x04_P3.96mm_Vertical, B.Cu at (89.3, 53.8)
- moved C289 75.5 mm to (99.9, 55.3), turned to 90 degrees
- moved C249 34.2 mm to (192.4, 140.5)
- moved C273 34.2 mm to (192.4, 148.7)
- moved C10 34.2 mm to (198.7, 153.9)
- moved C101 34.2 mm to (138.2, 91.2)
- moved C105 34.2 mm to (192.4, 90.9)
- moved C106 34.2 mm to (198.7, 120.9)
- moved C108 34.2 mm to (225.6, 121.0)
- moved C113 34.2 mm to (138.2, 94.7)
- moved C117 34.2 mm to (192.4, 94.4)
- moved C118 34.2 mm to (198.7, 117.5)
- moved C12 34.2 mm to (225.6, 154.0)
- moved C120 34.2 mm to (225.6, 117.5)
- moved C125 34.2 mm to (138.2, 99.4)
- moved C129 34.2 mm to (192.4, 99.2)
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Routing:
- net +5V: track 2034.9 -> 2099.6 mm
- net /C_Key/DIN: track 5.07 -> 6.97 mm
Other:
- board size 164 x 105 mm -> 164.1 x 109.9 mm
