File: Chromesthesia.kicad_pcb (KiCad board)
At the start: 2 copper layers, 164.1 x 109.9 mm, 582 parts, among them J3 Interface

Commit message: Text Added Production
Other:
- board text added: "CHROMESTHESIA"
- board text added: "EE496 - Bradley Miller, Kenny Yadav, Paolo Bahrami"
