File: Chromesthesia.kicad_sch (KiCad schematic)
At the start: 0 parts

Commit message: Schematic
Parts:
- added C289: 1000µF, Capacitor_THT:CP_Radial_D10.0mm_P5.00mm, symbol Device:C_Polarized
- added J1: Data In, symbol Connector_Generic:Conn_01x02
- added J2: Power In, symbol Connector_Generic:Conn_01x02
Connections:
- new net +5V: C289.1, J2.2 (Pin_2)
- new net C_Key/DIN: J1.2 (Pin_2)
- new net GND: C289.2, J1.1 (Pin_1), J2.1 (Pin_1)
- no-connect marks 0 -> 1
Other:
- added sheet A_Key (key.kicad_sch)
- added sheet As_Key (key.kicad_sch)
- added sheet B_Key (key.kicad_sch)
- added sheet C_Key (key.kicad_sch)
- added sheet Cs_Key (key.kicad_sch)
- added sheet D_Key (key.kicad_sch)
- added sheet Ds_Key (key.kicad_sch)
- added sheet E_Key (key.kicad_sch)
- added sheet F_Key (key.kicad_sch)
- added sheet Fs_Key (key.kicad_sch)
- added sheet G_Key (key.kicad_sch)
- added sheet Gs_Key (key.kicad_sch)

Commit message: Initial Production
Parts:
- removed J1: Data In, symbol Connector_Generic:Conn_01x02
- removed J2: Power In, symbol Connector_Generic:Conn_01x02
- added H1, H2, H3, H4: MountingHole, MountingHole:MountingHole_2.2mm_M2, symbol Mechanical:MountingHole
- added J3: Interface, Connector_JST:JST_VH_B4P-VH-FB-B_1x04_P3.96mm_Vertical, symbol Connector_Generic:Conn_01x04
Connections:
- net +5V: now also J3.1 (Pin_1)
- net C_Key/DIN: now also J3.4 (Pin_4)
- net GND: now also J3.2 (Pin_2), J3.3 (Pin_3)
Other:
- moved on the sheet: C289
